File: Schematics/BancoDePruebas/BancoDePruebas.kicad_pcb (KiCad board)
At the start: 2 copper layers, 81.1 x 69 mm, 55 parts, among them J1 LoadCell, J2 FROM_LIPO, J3 ALIM_ESC, J4 ESC_PWM_CONTROL, J5 H1, J6 H2, J7 UNA219_IF, J8 INA219_CURRENT, Q1 IRLML2502, Q2 IRF3808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

Commit message: Working ping back
Other:
- board text added: "@Spuertes @Araba_ST @vitorio08 @agambmel @bss_wrestling99 @pablunis_ @bern245 @red_ozon @zurano_"
- board text removed: "@Spuertes @Araba_ST @vitorio08 @agambmel"
Changed lines of the file:
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@@
     (fp_line (start 10.82 -1.72) (end 10.81641 -1.720064) (layer "F.SilkS") (width 0.12))
     (fp_line (start 3.582512 -2.207108) (end 3.861166 -1.890847) (layer "F.SilkS") (width 0.12))
-    (fp_arc (start 11.070011 -1.724215) (mid 11.102263 -1.900884) (end 11.194857 -2.054759) (layer "F.SilkS") (width 0.12))
-    (fp_arc (start 10.47 -2.369999) (mid 10.63682 -2.31867) (end 10.719999 -2.165211) (layer "F.SilkS") (width 0.12))
-    (fp_arc (start 11.316427 -1.7285) (mid 11.333055 -1.815275) (end 11.378833 -1.890847) (layer "F.SilkS") (width 0.12))
+    (fp_arc (start 11.070011 -1.724215) (mid 11.102268 -1.900879) (end 11.194857 -2.054759) (layer "F.SilkS") (width 0.12))
+    (fp_arc (start 10.47 -2.369999) (mid 10.636848 -2.318676) (end 10.719999 -2.165211) (layer "F.SilkS") (width 0.12))
+    (fp_arc (start 11.316427 -1.7285) (mid 11.333049 -1.81528) (end 11.378833 -1.890847) (layer "F.SilkS") (width 0.12))
     (fp_arc (start 10.81641 -1.720063) (mid 10.74803 -1.750569) (end 10.719999 -1.82) (layer "F.SilkS") (width 0.12))
     (fp_arc (start 4.52 -1.819999) (mid 4.491968 -1.750569) (end 4.423589 -1.720064) (layer "F.SilkS") (width 0.12))
-    (fp_arc (start 10.47 -2.226605) (mid 10.636822 -2.175277) (end 10.719999 -2.021817) (layer "F.SilkS") (width 0.12))
+    (fp_arc (start 10.47 -2.226605) (mid 10.63685 -2.175282) (end 10.719999 -2.021817) (layer "F.SilkS") (width 0.12))
     (fp_arc (start 4.52 -2.021818) (mid 4.603194 -2.175246) (end 4.77 -2.226605) (layer "F.SilkS") (width 0.12))
-    (fp_arc (start 3.861166 -1.890847) (mid 3.906978 -1.815287) (end 3.923572 -1.7285) (layer "F.SilkS") (width 0.12))
+    (fp_arc (start 3.861166 -1.890847) (mid 3.906966 -1.815286) (end 3.923572 -1.7285) (layer "F.SilkS") (width 0.12))
     (fp_arc (start 4.519999 -2.165212) (mid 4.60319 -2.318647) (end 4.77 -2.37) (layer "F.SilkS") (width 0.12))
     (fp_arc (start 4.045142 -2.054759) (mid 4.137725 -1.90088) (end 4.169988 -1.724215) (layer "F.SilkS") (width 0.12))
@@
   )
   (gr_line (start 116.45 116.9) (end 116.55 105.6) (layer "F.SilkS") (width 0.15))
-  (gr_line (start 119.3 96.7) (end 132.6 96.7) (layer "F.SilkS") (width 0.15))
+  (gr_line (start 118.45 96.85) (end 131.75 96.85) (layer "F.SilkS") (width 0.15))
   (gr_line (start 95.75 116.9) (end 116.45 116.9) (layer "F.SilkS") (width 0.15))
   (gr_rect (start 53.1 49.7) (end 134.175 118.7) (layer "Edge.Cuts") (width 0.1) (fill none))
@@
     (effects (font (size 1 1) (thickness 0.15)))
   )
-  (gr_text "@Spuertes\n@Araba_ST\n@vitorio08\n@agambmel" (at 121.8 100.2) (layer "F.SilkS")
+  (gr_text "@Spuertes\n@Araba_ST\n@vitorio08\n@agambmel\n@bss_wrestling99\n@pablunis_\n@bern245\n@red_ozon\n@zurano_" (at 119.75 104.3) (layer "F.SilkS")
     (effects (font (size 1 1) (thickness 0.15)) (justify left))
   )
-  (gr_text "Gracias a:" (at 123.7 95.8) (layer "F.SilkS")
+  (gr_text "Gracias a:" (at 122.85 95.95) (layer "F.SilkS")
     (effects (font (size 1 1) (thickness 0.15)))
   )

Commit message: Changes in UI
Other:
- board text added: "@Spuertes @Araba_ST @vitorio08 @agambmel @bss_wrestling99 @pablunis_ @bern245 @red_ozon @zurano_ @carlosbetdev"
- board text removed: "@Spuertes @Araba_ST @vitorio08 @agambmel @bss_wrestling99 @pablunis_ @bern245 @red_ozon @zurano_"
Changed lines of the file:
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@@
       (layerselection 0x00010fc_ffffffff)
       (disableapertmacros false)
-      (usegerberextensions false)
+      (usegerberextensions true)
       (usegerberattributes true)
-      (usegerberadvancedattributes true)
-      (creategerberjobfile true)
+      (usegerberadvancedattributes false)
+      (creategerberjobfile false)
       (svguseinch false)
       (svgprecision 6)
@@
       (psa4output false)
       (plotreference true)
-      (plotvalue true)
+      (plotvalue false)
       (plotinvisibletext false)
       (sketchpadsonfab false)
-      (subtractmaskfromsilk false)
+      (subtractmaskfromsilk true)
       (outputformat 1)
       (mirror false)
       (drillshape 0)
       (scaleselection 1)
-      (outputdirectory "")
+      (outputdirectory "Gerbers")
     )
   )
@@
     (fp_line (start 1.6 -0.8) (end 1.6 0.8) (layer "F.Fab") (width 0.1))
     (fp_line (start -1.6 -0.8) (end 1.6 -0.8) (layer "F.Fab") (width 0.1))
-    (pad "1" smd roundrect (at -1.5625 0 270) (size 1.325 1.8) (layers "F.Cu" "F.Paste" "F.Mask") (roundrect_rratio 0.188679)
+    (pad "1" smd roundrect (at -1.5625 0 270) (size 1.325 1.8) (layers "F.Cu" "F.Paste" "F.Mask") (roundrect_rratio 0.1886792453)
       (net 44 "V_FEEDBACK") (pintype "passive"))
-    (pad "2" smd roundrect (at 1.5625 0 270) (size 1.325 1.8) (layers "F.Cu" "F.Paste" "F.Mask") (roundrect_rratio 0.188679)
+    (pad "2" smd roundrect (at 1.5625 0 270) (size 1.325 1.8) (layers "F.Cu" "F.Paste" "F.Mask") (roundrect_rratio 0.1886792453)
       (net 1 "LIPO_NEG") (pintype "passive"))
     (model "${KICAD6_3DMODEL_DIR}/Capacitor_SMD.3dshapes/C_1206_3216Metric.wrl"
@@
     (fp_line (start -1.6 0.8) (end -1.6 -0.8) (layer "F.Fab") (width 0.1))
     (fp_line (start 1.6 0.8) (end -1.6 0.8) (layer "F.Fab") (width 0.1))
-    (pad "1" smd roundrect (at -1.5625 0 90) (size 1.325 1.8) (layers "F.Cu" "F.Paste" "F.Mask") (roundrect_rratio 0.188679)
+    (pad "1" smd roundrect (at -1.5625 0 90) (size 1.325 1.8) (layers "F.Cu" "F.Paste" "F.Mask") (roundrect_rratio 0.1886792453)
       (net 62 "Net-(U6-Pad6)") (pintype "passive"))
-    (pad "2" smd roundrect (at 1.5625 0 90) (size 1.325 1.8) (layers "F.Cu" "F.Paste" "F.Mask") (roundrect_rratio 0.188679)
+    (pad "2" smd roundrect (at 1.5625 0 90) (size 1.325 1.8) (layers "F.Cu" "F.Paste" "F.Mask") (roundrect_rratio 0.1886792453)
       (net 1 "LIPO_NEG") (pintype "passive"))
     (model "${KICAD6_3DMODEL_DIR}/Capacitor_SMD.3dshapes/C_1206_3216Metric.wrl"
@@
     (fp_line (start -1.6 -0.8) (end 1.6 -0.8) (layer "F.Fab") (width 0.1))
     (fp_line (start 1.6 0.8) (end -1.6 0.8) (layer "F.Fab") (width 0.1))
-    (pad "1" smd roundrect (at -1.55 0 270) (size 1.3 1.75) (layers "F.Cu" "F.Paste" "F.Mask") (roundrect_rratio 0.192308)
+    (pad "1" smd roundrect (at -1.55 0 270) (size 1.3 1.75) (layers "F.Cu" "F.Paste" "F.Mask") (roundrect_rratio 0.1923076923)
       (net 22 "+5V") (pintype "passive"))
-    (pad "2" smd roundrect (at 1.55 0 270) (size 1.3 1.75) (layers "F.Cu" "F.Paste" "F.Mask") (roundrect_rratio 0.192308)
+    (pad "2" smd roundrect (at 1.55 0 270) (size 1.3 1.75) (layers "F.Cu" "F.Paste" "F.Mask") (roundrect_rratio 0.1923076923)
       (net 47 "Net-(D2-Pad2)") (pintype "passive"))
     (model "${KICAD6_3DMODEL_DIR}/Resistor_SMD.3dshapes/R_1206_3216Metric.wrl"
@@
     (fp_line (start -1.6 0.8) (end -1.6 -0.8) (layer "F.Fab") (width 0.1))
     (fp_line (start 1.6 -0.8) (end 1.6 0.8) (layer "F.Fab") (width 0.1))
-    (pad "1" smd roundrect (at -1.5625 0 180) (size 1.325 1.8) (layers "F.Cu" "F.Paste" "F.Mask") (roundrect_rratio 0.188679)
+    (pad "1" smd roundrect (at -1.5625 0 180) (size 1.325 1.8) (layers "F.Cu" "F.Paste" "F.Mask") (roundrect_rratio 0.1886792453)
       (net 22 "+5V") (pintype "passive"))
-    (pad "2" smd roundrect (at 1.5625 0 180) (size 1.325 1.8) (layers "F.Cu" "F.Paste" "F.Mask") (roundrect_rratio 0.188679)
+    (pad "2" smd roundrect (at 1.5625 0 180) (size 1.325 1.8) (layers "F.Cu" "F.Paste" "F.Mask") (roundrect_rratio 0.1886792453)
       (net 1 "LIPO_NEG") (pintype "passive"))
     (model "${KICAD6_3DMODEL_DIR}/Capacitor_SMD.3dshapes/C_1206_3216Metric.wrl"
@@
     (fp_arc (start 3.861166 -1.890847) (mid 3.906966 -1.815286) (end 3.923572 -1.7285) (layer "F.SilkS") (width 0.12))
     (fp_arc (start 4.519999 -2.165212) (mid 4.60319 -2.318647) (end 4.77 -2.37) (layer "F.SilkS") (width 0.12))
-    (fp_arc (start 4.045142 -2.054759) (mid 4.137725 -1.90088) (end 4.169988 -1.724215) (layer "F.SilkS") (width 0.12))
+    (fp_arc (start 4.045142 -2.054759) (mid 4.137732 -1.900877) (end 4.169988 -1.724215) (layer "F.SilkS") (width 0.12))
     (fp_line (start -1.8 -1.8) (end -1.8 50.06) (layer "F.CrtYd") (width 0.05))
     (fp_line (start 17.04 50.06) (end 13.44 50.06) (layer "F.CrtYd") (width 0.05))
@@
     (fp_line (start -1.6 -0.8) (end 1.6 -0.8) (layer "F.Fab") (width 0.1))
     (fp_line (start 1.6 0.8) (end -1.6 0.8) (layer "F.Fab") (width 0.1))
-    (pad "1" smd roundrect (at -1.55 0 270) (size 1.3 1.75) (layers "F.Cu" "F.Paste" "F.Mask") (roundrect_rratio 0.192308)
+    (pad "1" smd roundrect (at -1.55 0 270) (size 1.3 1.75) (layers "F.Cu" "F.Paste" "F.Mask") (roundrect_rratio 0.1923076923)
       (net 22 "+5V") (pintype "passive"))
-    (pad "2" smd roundrect (at 1.55 0 270) (size 1.3 1.75) (layers "F.Cu" "F.Paste" "F.Mask") (roundrect_rratio 0.192308)
+    (pad "2" smd roundrect (at 1.55 0 270) (size 1.3 1.75) (layers "F.Cu" "F.Paste" "F.Mask") (roundrect_rratio 0.1923076923)
       (net 45 "Net-(D1-Pad2)") (pintype "passive"))
     (model "${KICAD6_3DMODEL_DIR}/Resistor_SMD.3dshapes/R_1206_3216Metric.wrl"
@@
   )
   (gr_line (start 116.45 116.9) (end 116.55 105.6) (layer "F.SilkS") (width 0.15))
-  (gr_line (start 118.45 96.85) (end 131.75 96.85) (layer "F.SilkS") (width 0.15))
+  (gr_line (start 116.95 94.6) (end 130.25 94.6) (layer "F.SilkS") (width 0.15))
   (gr_line (start 95.75 116.9) (end 116.45 116.9) (layer "F.SilkS") (width 0.15))
   (gr_rect (start 53.1 49.7) (end 134.175 118.7) (layer "Edge.Cuts") (width 0.1) (fill none))
@@
     (effects (font (size 1 1) (thickness 0.15)))
   )
-  (gr_text "@Spuertes\n@Araba_ST\n@vitorio08\n@agambmel\n@bss_wrestling99\n@pablunis_\n@bern245\n@red_ozon\n@zurano_" (at 119.75 104.3) (layer "F.SilkS")
+  (gr_text "@Spuertes\n@Araba_ST\n@vitorio08\n@agambmel\n@bss_wrestling99\n@pablunis_\n@bern245\n@red_ozon\n@zurano_\n@carlosbetdev" (at 118.5 102.95) (layer "F.SilkS")
     (effects (font (size 1 1) (thickness 0.15)) (justify left))
   )
-  (gr_text "Gracias a:" (at 122.85 95.95) (layer "F.SilkS")
+  (gr_text "Gracias a:" (at 121.35 93.7) (layer "F.SilkS")
     (effects (font (size 1 1) (thickness 0.15)))
   )
