File: Schematics/BancoDePruebas/BancoDePruebas.kicad_sch (KiCad schematic)
At the start: 40 parts, among them J1 LoadCell, J2 FROM_LIPO, J3 ALIM_ESC, J4 ESC_PWM_CONTROL, J5 H1, J6 H2, J7 UNA219_IF, J8 INA219_CURRENT, Q1 IRLML2502, Q2 IRF3808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

Commit message: Changes in UI
Other:
- company: (none) -> LaboratorioGluon
- title: (none) -> Banco de Pruebas
Changed lines of the file:
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@@
 (kicad_sch (version 20211123) (generator eeschema)
   (paper "A4")
+  (title_block
+    (title "Banco de Pruebas")
+    (date "2022-11-13")
+    (company "LaboratorioGluon")
+  )
   (junction (at 225.425 102.87) (diameter 0) (color 0 0 0 0)
   )
